File: RC_car.kicad_sch (KiCad schematic)
At the start: 36 parts, among them J1 nRF24L01, J10 MP1584_5V_IN-, J11 MP1584_IN+, J12 MP1584_IN-, J13 MP1584_OUT-, J14 MP1584_OUT+, J2 MOTOR, J3 BATTERY_12V, J4 SERVO, J5 I2C, J7 MP1584_5V_IN+, J8 MP1584_5V_OUT+, J9 MP1584_5V_OUT-, U2 L298N, U3 LM2596T-5

Commit message: Assign preliminary footprints to all components
Preliminary — to be verified against physical parts after delivery:
- L1 (33uH inductor): diameter and lead pitch
- C1, C2, C6 (electrolytics): diameter and pitch
- J2, J3 (screw terminals): pitch (assumed 5.08mm)
Parts:
- C1, C2, C4, C6: footprint (none) -> Capacitor_THT:CP_Radial_D8.0mm_P3.50mm
- C3, C5, C7, C8: footprint (none) -> Capacitor_THT:C_Disc_D5.0mm_W2.5mm_P5.00mm
- D5, D6, D7, D8: footprint Diode_SMD:D_SMA -> Diode_THT:D_DO-201AD_P15.24mm_Horizontal
- J1: footprint (none) -> Connector_PinHeader_2.54mm:PinHeader_2x04_P2.54mm_Vertical
- J10, J11, J12, J13, J14, J7, J8, J9: footprint (none) -> Connector_PinHeader_2.54mm:PinHeader_1x01_P2.54mm_Vertical
- J2, J3: footprint (none) -> TerminalBlock_Phoenix:TerminalBlock_Phoenix_MPT-2.54mm_2pol_Vertical
- J4: footprint (none) -> Connector_PinHeader_2.54mm:PinHeader_1x03_P2.54mm_Vertical
- J5: footprint (none) -> Connector_PinHeader_2.54mm:PinHeader_1x04_P2.54mm_Vertical
- L1: footprint (none) -> Inductor_THT:L_Radial_D8.0mm_P5.00mm
- R1, R2, R3, R4, R5, R6: footprint (none) -> Resistor_THT:R_Axial_DIN0207_L6.3mm_D2.5mm_P10.16mm
- U3: footprint Package_TO_SOT_THT:TO-220-5_P3.4x3.7mm_StaggerOdd_Lead3.8mm_Vertical -> Package_TO_SOT_THT:TO-220-5_P3.4x3.7mm_StaggerEven_Lead4.58mm_Vertical
Connections:
- net +5V: now reaches A1.27 (+5V), C2.1, C3.1, J5.2 (Pin_2), L1.2, R5.1, R6.1, U2.9 (Vss), U3.4 (FB)
Changed lines of the file:
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@@
 	)
 	(junction
+		(at 148.59 29.21)
+		(diameter 0)
+		(color 0 0 0 0)
+	)
+	(junction
 		(at 30.48 102.87)
 		(diameter 0)
@@
 	(wire
 		(pts
+			(xy 148.59 29.21) (xy 153.67 29.21)
+		)
+		(stroke
+			(width 0)
+			(type default)
+		)
+	)
+	(wire
+		(pts
 			(xy 64.77 154.94) (xy 64.77 157.48)
 		)
@@
 	(wire
 		(pts
-			(xy 143.51 29.21) (xy 153.67 29.21)
+			(xy 143.51 29.21) (xy 148.59 29.21)
 		)
 		(stroke
@@
 			)
 		)
-		(property "Footprint" ""
+		(property "Footprint" "TerminalBlock_Phoenix:TerminalBlock_Phoenix_MPT-2.54mm_2pol_Vertical"
 			(at 74.93 97.79 0)
 			(hide yes)
@@
 			)
 		)
-		(property "Footprint" ""
+		(property "Footprint" "Connector_PinHeader_2.54mm:PinHeader_1x01_P2.54mm_Vertical"
 			(at 121.92 81.28 0)
 			(hide yes)
@@
 			)
 		)
-		(property "Footprint" "Diode_SMD:D_SMA"
+		(property "Footprint" "Diode_THT:D_DO-201AD_P15.24mm_Horizontal"
 			(at 118.11 146.685 0)
 			(hide yes)
@@
 			)
 		)
-		(property "Footprint" ""
+		(property "Footprint" "Connector_PinHeader_2.54mm:PinHeader_1x01_P2.54mm_Vertical"
 			(at 121.92 71.12 0)
 			(hide yes)
@@
 			)
 		)
-		(property "Footprint" ""
+		(property "Footprint" "Resistor_THT:R_Axial_DIN0207_L6.3mm_D2.5mm_P10.16mm"
 			(at 206.502 53.34 90)
 			(hide yes)
@@
 			)
 		)
-		(property "Footprint" "Package_TO_SOT_THT:TO-220-5_P3.4x3.7mm_StaggerOdd_Lead3.8mm_Vertical"
+		(property "Footprint" "Package_TO_SOT_THT:TO-220-5_P3.4x3.7mm_StaggerEven_Lead4.58mm_Vertical"
 			(at 92.71 44.45 0)
 			(hide yes)
@@
 			)
 		)
-		(property "Footprint" ""
+		(property "Footprint" "Connector_PinHeader_2.54mm:PinHeader_1x01_P2.54mm_Vertical"
 			(at 82.55 110.49 0)
 			(hide yes)
@@
 			)
 		)
-		(property "Footprint" ""
+		(property "Footprint" "TerminalBlock_Phoenix:TerminalBlock_Phoenix_MPT-2.54mm_2pol_Vertical"
 			(at 129.54 152.4 0)
 			(hide yes)
@@
 			)
 		)
-		(property "Footprint" ""
+		(property "Footprint" "Connector_PinHeader_2.54mm:PinHeader_1x04_P2.54mm_Vertical"
 			(at 218.44 39.37 0)
 			(hide yes)
@@
 			)
 		)
-		(property "Footprint" "Diode_SMD:D_SMA"
+		(property "Footprint" "Diode_THT:D_DO-201AD_P15.24mm_Horizontal"
 			(at 107.95 184.785 0)
 			(hide yes)
@@
 			)
 		)
-		(property "Footprint" "Diode_SMD:D_SMA"
+		(property "Footprint" "Diode_THT:D_DO-201AD_P15.24mm_Horizontal"
 			(at 111.76 154.305 0)
 			(hide yes)
@@
 			)
 		)
-		(property "Footprint" ""
+		(property "Footprint" "Inductor_THT:L_Radial_D8.0mm_P5.00mm"
 			(at 120.65 29.21 0)
 			(hide yes)
@@
 			)
 		)
-		(property "Footprint" "Diode_SMD:D_SMA"
+		(property "Footprint" "Diode_THT:D_DO-201AD_P15.24mm_Horizontal"
 			(at 115.57 189.865 0)
 			(hide yes)
@@
 			)
 		)
-		(property "Footprint" ""
+		(property "Footprint" "Connector_PinHeader_2.54mm:PinHeader_1x01_P2.54mm_Vertical"
 			(at 82.55 95.25 0)
 			(hide yes)
@@
 			)
 		)
-		(property "Footprint" ""
+		(property "Footprint" "Resistor_THT:R_Axial_DIN0207_L6.3mm_D2.5mm_P10.16mm"
 			(at 57.912 119.38 90)
 			(hide yes)
@@
 			)
 		)
-		(property "Footprint" ""
+		(property "Footprint" "Resistor_THT:R_Axial_DIN0207_L6.3mm_D2.5mm_P10.16mm"
 			(at 129.032 76.2 90)
 			(hide yes)
@@
 			)
 		)
-		(property "Footprint" ""
+		(property "Footprint" "Connector_PinHeader_2.54mm:PinHeader_1x01_P2.54mm_Vertical"
 			(at 90.17 71.12 0)
 			(hide yes)
@@
 			)
 		)
-		(property "Footprint" ""
+		(property "Footprint" "Connector_PinHeader_2.54mm:PinHeader_1x01_P2.54mm_Vertical"
 			(at 123.19 110.49 0)
 			(hide yes)
@@
 			)
 		)
-		(property "Footprint" ""
+		(property "Footprint" "Capacitor_THT:C_Disc_D5.0mm_W2.5mm_P5.00mm"
 			(at 144.4752 44.45 0)
 			(hide yes)
@@
 			)
 		)
-		(property "Footprint" ""
+		(property "Footprint" "Capacitor_THT:CP_Radial_D8.0mm_P3.50mm"
 			(at 49.8348 54.61 0)
 			(hide yes)
@@
 			)
 		)
-		(property "Footprint" ""
+		(property "Footprint" "Resistor_THT:R_Axial_DIN0207_L6.3mm_D2.5mm_P10.16mm"
 			(at 79.502 181.61 90)
 			(hide yes)
@@
 			)
 		)
-		(property "Footprint" ""
+		(property "Footprint" "Connector_PinHeader_2.54mm:PinHeader_1x01_P2.54mm_Vertical"
 			(at 123.19 95.25 0)
 			(hide yes)
@@
 			)
 		)
-		(property "Footprint" ""
+		(property "Footprint" "Capacitor_THT:C_Disc_D5.0mm_W2.5mm_P5.00mm"
 			(at 134.62 64.4652 0)
 			(hide yes)
@@
 			)
 		)
-		(property "Footprint" ""
+		(property "Footprint" "Connector_PinHeader_2.54mm:PinHeader_2x04_P2.54mm_Vertical"
 			(at 149.86 73.66 0)
 			(hide yes)
@@
 			)
 		)
-		(property "Footprint" ""
+		(property "Footprint" "Connector_PinHeader_2.54mm:PinHeader_1x03_P2.54mm_Vertical"
 			(at 148.59 101.6 0)
 			(hide yes)
@@
 			)
 		)
-		(property "Footprint" ""
+		(property "Footprint" "Capacitor_THT:C_Disc_D5.0mm_W2.5mm_P5.00mm"
 			(at 70.8152 185.42 0)
 			(hide yes)
@@
 	)
 	(symbol
+		(lib_id "power:+5V")
+		(at 148.59 29.21 0)
+		(unit 1)
+		(body_style 1)
+		(exclude_from_sim no)
+		(in_bom yes)
+		(on_board yes)
+		(in_pos_files yes)
+		(dnp no)
+		(fields_autoplaced yes)
+		(property "Reference" "#PWR05"
+			(at 148.59 33.02 0)
+			(hide yes)
+			(show_name no)
+			(do_not_autoplace no)
+			(effects
+				(font
+					(size 1.27 1.27)
+				)
+			)
+		)
+		(property "Value" "+5V"
+			(at 148.59 24.13 0)
+			(show_name no)
+			(do_not_autoplace no)
+			(effects
+				(font
+					(size 1.27 1.27)
+				)
+			)
+		)
+		(property "Footprint" ""
+			(at 148.59 29.21 0)
+			(hide yes)
+			(show_name no)
+			(do_not_autoplace no)
+			(effects
+				(font
+					(size 1.27 1.27)
+				)
+			)
+		)
+		(property "Datasheet" ""
+			(at 148.59 29.21 0)
+			(hide yes)
+			(show_name no)
+			(do_not_autoplace no)
+			(effects
+				(font
+					(size 1.27 1.27)
+				)
+			)
+		)
+		(property "Description" "Power symbol creates a global label with name \"+5V\""
+			(at 148.59 29.21 0)
+			(hide yes)
+			(show_name no)
+			(do_not_autoplace no)
+			(effects
+				(font
+					(size 1.27 1.27)
+				)
+			)
+		)
+		(pin "1"
+		)
+		(instances
+			(project "RC_car"
+				(path "/b25f26a0-0a02-4673-8add-5c3f65c17eda"
+					(reference "#PWR05")
+					(unit 1)
+				)
+			)
+		)
+	)
+	(symbol
 		(lib_id "Device:C")
 		(at 49.53 118.11 0)
@@
 			)
 		)
-		(property "Footprint" ""
+		(property "Footprint" "Capacitor_THT:C_Disc_D5.0mm_W2.5mm_P5.00mm"
 			(at 50.4952 121.92 0)
 			(hide yes)
@@
 			)
 		)
-		(property "Footprint" ""
+		(property "Footprint" "Capacitor_THT:CP_Radial_D8.0mm_P3.50mm"
 			(at 142.24 54.9148 0)
 			(hide yes)
@@
 			)
 		)
-		(property "Footprint" ""
+		(property "Footprint" "Resistor_THT:R_Axial_DIN0207_L6.3mm_D2.5mm_P10.16mm"
 			(at 57.912 107.95 90)
 			(hide yes)
@@
 			)
 		)
-		(property "Footprint" ""
+		(property "Footprint" "Capacitor_THT:CP_Radial_D8.0mm_P3.50mm"
 			(at 21.2852 102.87 0)
 			(hide yes)
@@
 			)
 		)
-		(property "Footprint" ""
+		(property "Footprint" "Connector_PinHeader_2.54mm:PinHeader_1x01_P2.54mm_Vertical"
 			(at 90.17 81.28 0)
 			(hide yes)
@@
 			)
 		)
-		(property "Footprint" ""
+		(property "Footprint" "Resistor_THT:R_Axial_DIN0207_L6.3mm_D2.5mm_P10.16mm"
 			(at 201.422 45.72 90)
 			(hide yes)
@@
 			)
 		)
-		(property "Footprint" ""
+		(property "Footprint" "Capacitor_THT:CP_Radial_D8.0mm_P3.50mm"
 			(at 134.3152 44.45 0)
 			(hide yes)

Commit message: Change footprints J2/J3 to TerminalBlock_ARK-2P_P5.00mm
Parts:
- J2, J3: footprint TerminalBlock_Phoenix:TerminalBlock_Phoenix_MPT-2.54mm_2pol_Vertical -> TerminalBlock:TerminalBlock_ARK-2P_P5.00mm
Changed lines of the file:
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@@
 			)
 		)
-		(property "Footprint" "TerminalBlock_Phoenix:TerminalBlock_Phoenix_MPT-2.54mm_2pol_Vertical"
+		(property "Footprint" "TerminalBlock:TerminalBlock_ARK-2P_P5.00mm"
 			(at 74.93 97.79 0)
 			(hide yes)
@@
 			)
 		)
-		(property "Footprint" "TerminalBlock_Phoenix:TerminalBlock_Phoenix_MPT-2.54mm_2pol_Vertical"
+		(property "Footprint" "TerminalBlock:TerminalBlock_ARK-2P_P5.00mm"
 			(at 129.54 152.4 0)
 			(hide yes)

Commit message: Fix footprint names for R1-R6, L1, U3, J2, J3, J1 pin mapping
Parts:
- J2, J3: footprint TerminalBlock:TerminalBlock_ARK-2P_P5.00mm -> TerminalBlock_RND:TerminalBlock_RND_205-00001_1x02_P5.00mm_Horizontal
- L1: footprint Inductor_THT:L_Radial_D8.0mm_P5.00mm -> Inductor_THT:L_Radial_D8.7mm_P5.00mm_Fastron_07HCP
- R1, R2, R3, R4, R5, R6: footprint Resistor_THT:R_Axial_DIN0207_L6.3mm_D2.5mm_P10.16mm -> Resistor_THT:R_Axial_DIN0207_L6.3mm_D2.5mm_P10.16mm_Horizontal
- U3: footprint Package_TO_SOT_THT:TO-220-5_P3.4x3.7mm_StaggerEven_Lead4.58mm_Vertical -> Package_TO_SOT_THT:TO-220-5_P3.4x3.7mm_StaggerEven_Lead3.8mm_Vertical
Connections:
- net GND: now also J1.1 (Pin_a1); no longer J1.a1 (Pin_a1)
- net at C4.1, C5.2, J14.1 (Pin_1)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: now also J1.5 (Pin_b1); no longer J1.b1 (Pin_b1)
- net at A1.12 (D9): now also J1.2 (Pin_a2); no longer J1.a2 (Pin_a2)
- net at A1.13 (D10): now also J1.6 (Pin_b2); no longer J1.b2 (Pin_b2)
- net at A1.14 (D11): now also J1.7 (Pin_b3); no longer J1.b3 (Pin_b3)
- net at A1.15 (D12): now also J1.4 (Pin_a4); no longer J1.a4 (Pin_a4)
- net at A1.16 (D13): now also J1.3 (Pin_a3); no longer J1.a3 (Pin_a3)
Changed lines of the file:
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@@
 			)
 		)
-		(property "Footprint" "TerminalBlock:TerminalBlock_ARK-2P_P5.00mm"
+		(property "Footprint" "TerminalBlock_RND:TerminalBlock_RND_205-00001_1x02_P5.00mm_Horizontal"
 			(at 74.93 97.79 0)
 			(hide yes)
@@
 			)
 		)
-		(property "Footprint" "Resistor_THT:R_Axial_DIN0207_L6.3mm_D2.5mm_P10.16mm"
+		(property "Footprint" "Resistor_THT:R_Axial_DIN0207_L6.3mm_D2.5mm_P10.16mm_Horizontal"
 			(at 206.502 53.34 90)
 			(hide yes)
@@
 			)
 		)
-		(property "Footprint" "Package_TO_SOT_THT:TO-220-5_P3.4x3.7mm_StaggerEven_Lead4.58mm_Vertical"
+		(property "Footprint" "Package_TO_SOT_THT:TO-220-5_P3.4x3.7mm_StaggerEven_Lead3.8mm_Vertical"
 			(at 92.71 44.45 0)
 			(hide yes)
@@
 			)
 		)
-		(property "Footprint" "TerminalBlock:TerminalBlock_ARK-2P_P5.00mm"
+		(property "Footprint" "TerminalBlock_RND:TerminalBlock_RND_205-00001_1x02_P5.00mm_Horizontal"
 			(at 129.54 152.4 0)
 			(hide yes)
@@
 			)
 		)
-		(property "Footprint" "Inductor_THT:L_Radial_D8.0mm_P5.00mm"
+		(property "Footprint" "Inductor_THT:L_Radial_D8.7mm_P5.00mm_Fastron_07HCP"
 			(at 120.65 29.21 0)
 			(hide yes)
@@
 			)
 		)
-		(property "Footprint" "Resistor_THT:R_Axial_DIN0207_L6.3mm_D2.5mm_P10.16mm"
+		(property "Footprint" "Resistor_THT:R_Axial_DIN0207_L6.3mm_D2.5mm_P10.16mm_Horizontal"
 			(at 57.912 119.38 90)
 			(hide yes)
@@
 			)
 		)
-		(property "Footprint" "Resistor_THT:R_Axial_DIN0207_L6.3mm_D2.5mm_P10.16mm"
+		(property "Footprint" "Resistor_THT:R_Axial_DIN0207_L6.3mm_D2.5mm_P10.16mm_Horizontal"
 			(at 129.032 76.2 90)
 			(hide yes)
@@
 			)
 		)
-		(property "Footprint" "Resistor_THT:R_Axial_DIN0207_L6.3mm_D2.5mm_P10.16mm"
+		(property "Footprint" "Resistor_THT:R_Axial_DIN0207_L6.3mm_D2.5mm_P10.16mm_Horizontal"
 			(at 79.502 181.61 90)
 			(hide yes)
@@
 			)
 		)
-		(pin "a1"
+		(pin "6"
 		)
-		(pin "b3"
+		(pin "1"
 		)
-		(pin "b1"
+		(pin "2"
 		)
-		(pin "a2"
+		(pin "5"
 		)
-		(pin "a4"
+		(pin "4"
 		)
-		(pin "b4"
+		(pin "3"
 		)
-		(pin "a3"
+		(pin "8"
 		)
-		(pin "b2"
+		(pin "7"
 		)
 		(instances
@@
 			)
 		)
-		(property "Footprint" "Resistor_THT:R_Axial_DIN0207_L6.3mm_D2.5mm_P10.16mm"
+		(property "Footprint" "Resistor_THT:R_Axial_DIN0207_L6.3mm_D2.5mm_P10.16mm_Horizontal"
 			(at 57.912 107.95 90)
 			(hide yes)
@@
 			)
 		)
-		(property "Footprint" "Resistor_THT:R_Axial_DIN0207_L6.3mm_D2.5mm_P10.16mm"
+		(property "Footprint" "Resistor_THT:R_Axial_DIN0207_L6.3mm_D2.5mm_P10.16mm_Horizontal"
 			(at 201.422 45.72 90)
 			(hide yes)

Commit message: PCB routing: power rails and I2C/signal traces
Parts:
- C1, C2, C3, C4, C5, C6, C7, C8: KiLib_Generator (none) -> capacitor/THT/other
- D1, D5, D6, D7, D8: KiLib_Generator (none) -> diode/THT
- J1, J10, J11, J12, J13, J14, J4, J5, J7, J8, J9: KiLib_Generator (none) -> connector/pin_header_socket
- J2, J3: KiLib_Generator (none) -> terminal_block/RND
- L1: KiLib_Generator (none) -> choke_THT
- R1, R2, R3, R4, R5, R6: KiLib_Generator (none) -> resistor/THT
- U2, U3: KiLib_Generator (none) -> package/TO_SOT/THT
